File: kiCad/temp_vibe_board/temp_vibe_board/temp_vibe_board.kicad_pcb (KiCad board)
At the start: 2 copper layers, 63 x 85.3 mm, 20 parts, among them J1 VDD, J2 GND, J3 SDA, J4 SCL, J5 VDD, J6 GND, J7 SDA2, J8 SCL2, J9 Conn_01x02_Pin, U1 DEV-13907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

Commit message: updated_temp_vibe_board
Parts:
- removed J2, J6: GND, Connector_PinHeader_2.54mm:PinHeader_1x01_P2.54mm_Horizontal
- removed J3: SDA, Connector_PinHeader_2.54mm:PinHeader_1x01_P2.54mm_Horizontal
- removed J4: SCL, Connector_PinHeader_2.54mm:PinHeader_1x01_P2.54mm_Horizontal
- removed J5: VDD, Connector_PinHeader_2.54mm:PinHeader_1x01_P2.54mm_Horizontal
- removed J7: SDA2, Connector_PinHeader_2.54mm:PinHeader_1x01_P2.54mm_Horizontal
- removed J8: SCL2, Connector_PinHeader_2.54mm:PinHeader_1x01_P2.54mm_Horizontal
- J1: value VDD -> Conn_01x04_Pin; footprint Connector_PinHeader_2.54mm:PinHeader_1x01_P2.54mm_Horizontal -> Connector_PinHeader_2.54mm:PinHeader_1x04_P2.54mm_Horizontal
- J9: value Conn_01x02_Pin -> Conn_01x04_Pin; footprint Connector_JST:JST_EH_S2B-EH_1x02_P2.50mm_Horizontal -> Connector_PinHeader_2.54mm:PinHeader_1x04_P2.54mm_Horizontal
- moved J9 48.5 mm to (79.4, 32.5), turned to 0 degrees
- moved J1 48.3 mm to (31.4, 40.1), turned to 180 degrees
Connections:
- U1 pad J1_11: MCUINT1 -> unconnected-(U1-DAC2/ADC2_9/GPIO26/26-PadJ1_11)
- U1 pad J2_12: MCUINT2 -> unconnected-(U1-V_SPI_CS0/LED(BLUE)/GPIO5/5-PadJ2_12)
- U2 pad 12: MCUINT1 -> unconnected-(U2-INT-Pad12)
- U3 pad 12: MCUINT2 -> unconnected-(U3-INT-Pad12)
Routing:
- net VDDIO: track 170.9 -> 209.6 mm, vias 5 -> 7
- net MCUINT1: track 25.6 -> 0.00 mm, vias 2 -> 0
- net MCUINT2: track 19.5 -> 0.00 mm, vias 1 -> 0
- net SCL: track 39.2 -> 31.6 mm
- net Net-(U2-AD0/MISO): track 0.00 -> 3.57 mm, vias 0 -> 2
- net GND: track 11.3 -> 7.78 mm, vias 0 -> 5
- net SDA2: track 55.1 -> 56.0 mm
- net SDA: vias 4 -> 5
Other:
- board size 63 x 85.3 mm -> 63.1 x 97.5 mm

Commit message: MPU6050 PCB
Parts:
- removed C1, C2, C3, C4: 0.1 uF, Capacitor_SMD:C_0805_2012Metric
- removed U2, U3: MPU-9250, Sensor_Motion:InvenSense_QFN-24_3x3mm_P0.4mm
- added C5: 0.1 uF, Capacitor_SMD:C_0805_2012Metric, F.Cu at (120.5, 93.5)
- added C6: 0.1 uF, Capacitor_SMD:C_0805_2012Metric, F.Cu at (120.5, 96.5)
- added C7: 0.1 uF, Capacitor_SMD:C_0805_2012Metric, F.Cu at (167.0, 83.0)
- added C8: 0.1 uF, Capacitor_SMD:C_0805_2012Metric, F.Cu at (167.0, 86.0)
- added U4: MPU-6050, Sensor_Motion:InvenSense_QFN-24_4x4mm_P0.5mm, F.Cu at (118.8, 77.0)
- added U5: MPU-6050, Sensor_Motion:InvenSense_QFN-24_4x4mm_P0.5mm, F.Cu at (169.1, 73.8)
- moved R3 91.8 mm to (126.4, 90.6)
- moved J9 91.8 mm to (167.7, 57.5)
- moved U1 91.8 mm to (143.4, 84.3)
- moved J1 91.8 mm to (119.7, 65.2)
- moved R1 91.8 mm to (160.3, 76.8)
- moved R2 91.8 mm to (160.3, 70.9)
- moved R4 91.8 mm to (125.4, 76.1)
Routing:
- net GND: track 7.78 -> 240.9 mm, vias 5 -> 15
- net Net-(U4-CPOUT): track 0.00 -> 32.0 mm, vias 0 -> 2
- net Net-(U5-CPOUT): track 0.00 -> 31.9 mm, vias 0 -> 2
- net VDDIO: track 209.6 -> 194.3 mm, vias 7 -> 4
- net SCL2: track 57.8 -> 49.2 mm, vias 0 -> 4
- net SDA: track 37.0 -> 28.8 mm, vias 5 -> 3
- net Net-(U2-REGOUT): track 5.34 -> 0.00 mm
- net Net-(U3-REGOUT): track 3.67 -> 0.00 mm, vias 2 -> 0
- net Net-(U2-AD0/MISO): track 3.57 -> 0.00 mm, vias 2 -> 0
- net SDA2: track 56.0 -> 58.0 mm, vias 4 -> 2
- net SCL: track 31.6 -> 30.4 mm, vias 0 -> 2
Other:
- outline, holes or cut-outs redrawn
- board text removed: "MPU"
